Commit message: valkyrie model added

File: cpp/Draco/RobotModel/draco.urdf (robot description, URDF)
Before this commit: robot draco, 9 links, 8 joints
Links:
- removed link FootInBack
- removed link FootInFront
- removed link FootOutBack
- removed link FootOutFront
Joints:
- removed joint foot_Offset1
- removed joint foot_Offset2
- removed joint foot_Offset3
- removed joint foot_Offset4
- joint ground_joint: origin xyz=0 0 2.0 rpy=0 0 0 -> xyz=0 0 0 rpy=0 0 0
