Commit message: debuging urdf

File: cpp/Draco/RobotModel/mk_draco.urdf (robot description, URDF)
Before this commit: robot draco, 5 links, 4 joints
Joints:
- joint ankle: origin xyz=0 0 -0.49 rpy=0.0 0.0 0.0 -> xyz=0 0.0 -0.36 rpy=0.0 0.0 0.0
- joint kneePitch: origin xyz=0 0 -0.49 rpy=0.0 0.0 0.0 -> xyz=0 -0.00 -0.494 rpy=0.0 0.0 0.0
